Commit message: V1

File: franka_description/robots/panda_arm.xacro (robot description, xacro)
@@ -307,5 +307,5 @@
     <joint name="${arm_id}_joint8" type="fixed">
       <!--origin rpy="0 0 0" xyz="0 0 0.107"/-->
-      <origin rpy="0 0 0" xyz="0 0 0.232"/>
+      <origin rpy="0 0 0" xyz="0 0 0.257"/> <!-- panda_joint8 위치를 default에 대해 15cm offset -->
       <parent link="${arm_id}_link7"/>
       <child link="${arm_id}_link8"/>

File: franka_robotiq_description/urdf/robot.urdf.xacro (robot description, xacro)
@@ -24,5 +24,5 @@
   <!-- connection between panda arm and robotiq gripper -->
   <!-- origin xyz="0 0 0" rpy="0 0 -1.570796" / -->
-  <origin xyz="0 0 -0.125" rpy="0 0 -1.570796" />
+  <origin xyz="0 0 -0.15" rpy="0 0 -1.570796" /> <!-- panda_joint8 위치 offset에 대해 역방향으로 15cm 보정 -->
     </xacro:robotiq_gripper>
   </xacro:if>

Commit message: teleop

File: franka_description/robots/panda_arm.xacro (robot description, xacro)
@@ -306,6 +306,7 @@
     </link>
     <joint name="${arm_id}_joint8" type="fixed">
-      <!--origin rpy="0 0 0" xyz="0 0 0.107"/-->
-      <origin rpy="0 0 0" xyz="0 0 0.257"/> <!-- panda_joint8 위치를 default에 대해 15cm offset -->
+      <!-- <origin rpy="0 0 0" xyz="0 0 0.107"/> -->
+      <!-- panda_joint8 위치를 default에 대해 15cm offset -->
+      <origin rpy="0 0 0" xyz="0 0 0.257"/>
       <parent link="${arm_id}_link7"/>
       <child link="${arm_id}_link8"/>

File: franka_robotiq_description/urdf/robot.urdf.xacro (robot description, xacro)
@@ -22,7 +22,8 @@
     <xacro:include filename="$(find robotiq_description)/urdf/robotiq_2f_85_macro.urdf.xacro"/>
     <xacro:robotiq_gripper name="RobotiqGripperHardwareInterface" prefix="" parent="$(arg arm_id)_link8" use_fake_hardware="$(arg use_fake_hardware)" fake_sensor_commands="$(arg fake_sensor_commands)" include_ros2_control="false">
-  <!-- connection between panda arm and robotiq gripper -->
-  <!-- origin xyz="0 0 0" rpy="0 0 -1.570796" / -->
-  <origin xyz="0 0 -0.15" rpy="0 0 -1.570796" /> <!-- panda_joint8 위치 offset에 대해 역방향으로 15cm 보정 -->
+	  <!-- connection between panda arm and robotiq gripper -->
+    <!-- <origin xyz="0 0 0" rpy="0 0 -1.570796"/> -->
+  <!-- panda_joint8 위치 offset에 대해 역방향으로 15cm 보정 -->
+      <origin xyz="0 0 -0.15" rpy="0 0 -1.570796"/>
     </xacro:robotiq_gripper>
   </xacro:if>
